File: peripherals.kicad_sch (KiCad schematic)
At the start: 0 parts

Commit message: feat(power & programmer): Finished Schematic building. Now sourcing for parts.
Parts:
- added C10, C11, C8, C9: 390nF, symbol Device:C_Small
- added C57: 2.2nF, symbol Device:C_Small
- added C58, C60: 0.1uF, symbol Device:C_Small
- added C59: 10nF, symbol Device:C_Small
- added C6, C7: 100nF, symbol Device:C_Small
- added J1, J2, J3, J4, J5, J6: HCTL HC-5264-3A, Connector_PinHeader_2.54mm:HC-5264-3A, symbol Connector:HCTL_HC-5264-3A
- added R36, R37: 4.7kΩ, symbol Device:R_Small_US
- added SN74LVC2G1: (no value), Package_SO:VSSOP-8_3x3mm_P0.65mm, symbol 74xGxx:SN74LVC2G241
- added SW1, SW2, SW3, SW4, SW5, SW6: SW_Push, symbol Switch:SW_Push
- added U9: MPU-6050, Sensor_Motion:InvenSense_QFN-24_4x4mm_P0.5mm, symbol Sensor_Motion:MPU-6050
Connections:
- new net: C57.1, U9.20 (CPOUT)
- new net: C58.2, U9.10 (REGOUT)
- new net +7V4A: J1.2 (Pin_2), J2.2 (Pin_2)
- new net +7V4B: J3.2 (Pin_2), J4.2 (Pin_2)
- new net +7V4C: J5.2 (Pin_2), J6.2 (Pin_2)
- new net +ESP_3.3V: C59.1, C60.2, R36.1, R37.1, SN74LVC2G1.8 (VCC), U9.13 (VDD), U9.8 (VLOGIC)
- new net DATA: J1.1 (Pin_1), J2.1 (Pin_1), J3.1 (Pin_1), J4.1 (Pin_1), J5.1 (Pin_1), J6.1 (Pin_1), SN74LVC2G1.2 (1A), SN74LVC2G1.3 (2Y)
- new net GND: C10.2, C11.2, C57.2, C58.1, C59.2, C6.2, C60.1, C7.2, C8.2, C9.2, J1.3 (Pin_3), J2.3 (Pin_3), J3.3 (Pin_3), J4.3 (Pin_3), J5.3 (Pin_3), J6.3 (Pin_3), SN74LVC2G1.4 (GND), SW1.1, SW2.1, SW3.1, SW4.1, SW5.1, SW6.1, U9.1 (CLKIN), U9.11 (FSYNC), U9.18 (GND), U9.9 (AD0)
- new net I2C_SCL: R37.2, U9.23 (SCL)
- new net I2C_SDA: R36.2, U9.24 (SDA)
- new net SERVO_DIR: SN74LVC2G1.1 (~1OE), SN74LVC2G1.7 (2OE)
- new net SERVO_RX: SN74LVC2G1.6 (1Y)
- new net SERVO_TX: SN74LVC2G1.5 (2A)
- new net SWITCH_0: C6.1, SW1.2
- new net SWITCH_1: C7.1, SW2.2
- new net SWITCH_2: C8.1, SW3.2
- new net SWITCH_3: C9.1, SW4.2
- new net SWITCH_4: C10.1, SW5.2
- new net SWITCH_5: C11.1, SW6.2
- no-connect marks 0 -> 3
